File: circuit/sega.sch (EAGLE design)
At the start: 1 part

Commit message: Update circuit design to v1.2
 - Raspberry Pi Zero mounted directly to the board replaces header
 - DB9 connectors replace individual jumper wires to the controller
Parts:
- removed GPIO: (no value), pinhead:PINHD-2X13
- added PI: PIZERO_THROUGH_HOLE, pizero:PIZERO_THROUGH_HOLE
Connections:
- net N$1: now also PI.11; no longer GPIO.11
- net N$10: now also PI.8; no longer GPIO.8
- net N$11: now also PI.10; no longer GPIO.10
- net N$12: now also PI.12; no longer GPIO.12
- net N$13: now also PI.16; no longer GPIO.16
- net N$14: now also PI.18; no longer GPIO.18
- net N$15: now also PI.22; no longer GPIO.22
- net N$16: now also PI.24; no longer GPIO.24
- net N$17: now also PI.26; no longer GPIO.26
- net N$2: now also PI.14, PI.20, PI.25, PI.6, PI.9; no longer GPIO.14, GPIO.20, GPIO.25, GPIO.6, GPIO.9
- net N$3: now also PI.13; no longer GPIO.13
- net N$4: now also PI.3; no longer GPIO.3
- net N$5: now also PI.5; no longer GPIO.5
- net N$6: now also PI.7; no longer GPIO.7
- net N$7: now also PI.15; no longer GPIO.15
- net N$8: now also PI.19; no longer GPIO.19
- net N$9: now also PI.21; no longer GPIO.21
